File: PCB/Yari.kicad_pcb (KiCad board)
At the start: 2 copper layers, 131.9 x 104.1 mm, 46 parts

Commit message: Updated render images and added gerber files
Routing:
- net middle_bottom: track 20.6 -> 21.1 mm

Commit message: Started over in Kicad
Parts:
- removed MCU1: , ceoloide:mcu_supermini_nrf52840
- removed MH1, MH2, MH3, MH4, MH5: , ceoloide:mounting_hole_npth
- removed PWR1: , ceoloide:power_switch_smd_side
- removed RST1: , ceoloide:reset_switch_smd_side
- added D19: ~, ScottoKeebs_Components:Diode_SOD-123, F.Cu at (131.4, 92.2)
- added D20: ~, ScottoKeebs_Components:Diode_SOD-123, B.Cu at (263.0, 98.5)
- added D21: ~, ScottoKeebs_Components:Diode_SOD-123, B.Cu at (243.9, 111.8)
- added D22: ~, ScottoKeebs_Components:Diode_SOD-123, B.Cu at (223.6, 120.9)
- added D23: ~, ScottoKeebs_Components:Diode_SOD-123, B.Cu at (205.6, 115.4)
- added D24: ~, ScottoKeebs_Components:Diode_SOD-123, B.Cu at (187.5, 113.3)
- added D25: ~, ScottoKeebs_Components:Diode_SOD-123, B.Cu at (260.6, 81.4)
- added D26: ~, ScottoKeebs_Components:Diode_SOD-123, B.Cu at (242.8, 95.9)
- added D27: ~, ScottoKeebs_Components:Diode_SOD-123, B.Cu at (223.7, 104.8)
- added D28: ~, ScottoKeebs_Components:Diode_SOD-123, B.Cu at (205.6, 99.6)
- added D29: ~, ScottoKeebs_Components:Diode_SOD-123, B.Cu at (187.6, 96.9)
- added D30: ~, ScottoKeebs_Components:Diode_SOD-123, B.Cu at (258.3, 65.2)
- added D31: ~, ScottoKeebs_Components:Diode_SOD-123, B.Cu at (241.4, 77.7)
- added D32: ~, ScottoKeebs_Components:Diode_SOD-123, B.Cu at (223.3, 87.3)
- added D33: ~, ScottoKeebs_Components:Diode_SOD-123, B.Cu at (205.4, 81.4)
- added D34: ~, ScottoKeebs_Components:Diode_SOD-123, B.Cu at (187.6, 79.1)
- added D35: ~, ScottoKeebs_Components:Diode_SOD-123, B.Cu at (193.6, 63.4)
- added D36: ~, ScottoKeebs_Components:Diode_SOD-123, B.Cu at (175.0, 57.8)
- added D37: ~, ScottoKeebs_Components:Diode_SOD-123, B.Cu at (158.0, 48.6)
- added D38: ~, ScottoKeebs_Components:Diode_SOD-123, B.Cu at (167.8, 76.6)
- added H1: ~, MountingHole:MountingHole_2.2mm_M2_DIN965, F.Cu at (23.4, 52.4)
- added H1: ~, MountingHole:MountingHole_2.2mm_M2_DIN965, F.Cu at (257.6, 112.0)
- added H10: ~, MountingHole:MountingHole_2.2mm_M2_DIN965, F.Cu at (197.1, 58.7)
- added H10: ~, MountingHole:MountingHole_2.2mm_M2_DIN965, F.Cu at (84.0, 105.7)
- added H2: ~, MountingHole:MountingHole_2.2mm_M2_DIN965, F.Cu at (94.9, 39.4)
- added H2: ~, MountingHole:MountingHole_2.2mm_M2_DIN965, F.Cu at (185.3, 125.5)
- added H3: ~, MountingHole:MountingHole_2.2mm_M2_DIN965, F.Cu at (55.4, 38.9)
- added H3: ~, MountingHole:MountingHole_2.2mm_M2_DIN965, F.Cu at (227.1, 126.1)
- added H4: ~, MountingHole:MountingHole_2.2mm_M2_DIN965, F.Cu at (25.2, 104.9)
- added H4: ~, MountingHole:MountingHole_2.2mm_M2_DIN965, F.Cu at (255.9, 59.5)
- added H5: ~, MountingHole:MountingHole_2.2mm_M2_DIN965, F.Cu at (156.7, 63.6)
- added H5: ~, MountingHole:MountingHole_2.2mm_M2_DIN965, F.Cu at (124.4, 100.7)
- added H6: ~, MountingHole:MountingHole_2.2mm_M2_DIN965, F.Cu at (187.3, 89.5)
- added H6: ~, MountingHole:MountingHole_2.2mm_M2_DIN965, F.Cu at (221.5, 78.2)
- added H6: ~, MountingHole:MountingHole_2.2mm_M2_DIN965, F.Cu at (75.5, 66.8)
- added H6: ~, MountingHole:MountingHole_2.2mm_M2_DIN965, F.Cu at (61.1, 86.5)
- added H6: ~, MountingHole:MountingHole_2.2mm_M2_DIN965, F.Cu at (205.5, 91.9)
- added H6: ~, MountingHole:MountingHole_2.2mm_M2_DIN965, B.Cu at (148.1, 35.0)
- added H7: ~, MountingHole:MountingHole_2.2mm_M2_DIN965, F.Cu at (223.6, 97.3)
- added H7: ~, MountingHole:MountingHole_2.2mm_M2_DIN965, F.Cu at (56.6, 57.9)
- added H8: ~, MountingHole:MountingHole_2.2mm_M2_DIN965, F.Cu at (37.6, 70.1)
- added H8: ~, MountingHole:MountingHole_2.2mm_M2_DIN965, F.Cu at (242.8, 88.9)
- added H9: ~, MountingHole:MountingHole_2.2mm_M2_DIN965, F.Cu at (133.2, 129.2)
- added H9: ~, MountingHole:MountingHole_2.2mm_M2_DIN965, B.Cu at (93.5, 72.6)
- added J1: JST_CN, Connector_JST:JST_PH_S2B-PH-K_1x02_P2.00mm_Horizontal, F.Cu at (125.1, 78.9)
- added J2: JST_CN, Connector_JST:JST_PH_S2B-PH-K_1x02_P2.00mm_Horizontal, B.Cu at (156.1, 87.1)
- added REF**: mousebites 2mm, PCM_marbastlib-various:mousebites_2.5mm, F.Cu at (135.1, 78.2)
- added REF**: mousebites 2mm, PCM_marbastlib-various:mousebites_2.5mm, F.Cu at (146.0, 104.7)
- added REF**: mousebites 2mm, PCM_marbastlib-various:mousebites_2.5mm, F.Cu at (145.9, 87.1)
- added REF**: mousebites 2mm, PCM_marbastlib-various:mousebites_2.5mm, F.Cu at (135.1, 59.5)
- added REF**: mousebites 2mm, PCM_marbastlib-various:mousebites_2.5mm, F.Cu at (135.1, 96.4)
- added REF**: mousebites 2mm, PCM_marbastlib-various:mousebites_2.5mm, F.Cu at (145.9, 69.4)
- added S19: ~, ScottoKeebs_Hotswap:Hotswap_Choc_V1_1.00u, F.Cu at (122.4, 90.0)
- added S20: ~, ScottoKeebs_Hotswap:Hotswap_Choc_V1_1.00u, B.Cu at (254.3, 101.4)
- added S21: ~, ScottoKeebs_Hotswap:Hotswap_Choc_V1_1.00u, B.Cu at (235.0, 114.3)
- added S22: ~, ScottoKeebs_Hotswap:Hotswap_Choc_V1_1.00u, B.Cu at (214.5, 122.7)
- added S23: ~, ScottoKeebs_Hotswap:Hotswap_Choc_V1_1.00u, B.Cu at (196.5, 117.3)
- added S24: ~, ScottoKeebs_Hotswap:Hotswap_Choc_V1_1.00u, B.Cu at (178.5, 114.8)
- added S25: ~, ScottoKeebs_Hotswap:Hotswap_Choc_V1_1.00u, B.Cu at (252.0, 84.5)
- added S26: ~, ScottoKeebs_Hotswap:Hotswap_Choc_V1_1.00u, B.Cu at (233.8, 97.4)
- added S27: ~, ScottoKeebs_Hotswap:Hotswap_Choc_V1_1.00u, B.Cu at (214.5, 105.7)
- added S28: ~, ScottoKeebs_Hotswap:Hotswap_Choc_V1_1.00u, B.Cu at (196.5, 100.3)
- added S29: ~, ScottoKeebs_Hotswap:Hotswap_Choc_V1_1.00u, B.Cu at (178.5, 97.8)
- added S30: ~, ScottoKeebs_Hotswap:Hotswap_Choc_V1_1.00u, B.Cu at (249.6, 67.7)
- added S31: ~, ScottoKeebs_Hotswap:Hotswap_Choc_V1_1.00u, B.Cu at (232.6, 80.4)
- added S32: ~, ScottoKeebs_Hotswap:Hotswap_Choc_V1_1.00u, B.Cu at (214.5, 88.7)
- added S33: ~, ScottoKeebs_Hotswap:Hotswap_Choc_V1_1.00u, B.Cu at (196.5, 83.3)
- added S34: ~, ScottoKeebs_Hotswap:Hotswap_Choc_V1_1.00u, B.Cu at (178.5, 80.8)
- added S35: ~, ScottoKeebs_Hotswap:Hotswap_Choc_V1_1.00u, B.Cu at (184.5, 62.6)
- added S36: ~, ScottoKeebs_Hotswap:Hotswap_Choc_V1_1.00u, B.Cu at (166.1, 55.5)
- added S37: ~, ScottoKeebs_Hotswap:Hotswap_Choc_V1_1.00u, B.Cu at (149.6, 44.8)
- added SW1: SW_PS, PCM_marbastlib-various:SW_MSK12C02-HB, F.Cu at (132.2, 103.2)
- added SW2: SW_RST, Button_Switch_SMD:SW_SPST_B3U-1000P, F.Cu at (117.5, 77.7)
- added SW3: SW_PS, PCM_marbastlib-various:SW_MSK12C02-HB, B.Cu at (148.9, 61.2)
- added SW4: SW_RST, Button_Switch_SMD:SW_SPST_B3U-1000P, B.Cu at (163.6, 86.7)
- added SW5: RotaryEncoder_Switch, PCM_marbastlib-various:ROT_Alps_EC11E-Switch, B.Cu at (157.2, 74.0)
- added U1: Nice_Nano_V2, ScottoKeebs_MCU:Nice_Nano_V2_Flipped, F.Cu at (122.7, 58.8)
- added U2: Nice_Nano_V2, ScottoKeebs_MCU:Nice_Nano_V2_Flipped, B.Cu at (158.4, 105.5)
- D1, D10, D11, D12, D13, D14, D15, D16, D17, D18, D2, D3, D4, D5, D6, D7, D8, D9: value (none) -> ~; footprint ceoloide:diode_tht_sod123 -> ScottoKeebs_Components:Diode_SOD-123
- LED1: value (none) -> SK6812MINI-E; footprint ceoloide:led_SK6812mini-e (underglow, reversible) -> PCM_marbastlib-various:LED_6028R; moved to B.Cu
- LED2: value (none) -> SK6812MINI-E; footprint ceoloide:led_SK6812mini-e (underglow, reversible) -> PCM_marbastlib-various:LED_6028R
- S1, S10, S11, S12, S13, S14, S15, S16, S17, S18, S2, S3, S4, S5, S6, S7, S8, S9: value (none) -> ~; footprint ceoloide:switch_choc_v1_v2 -> ScottoKeebs_Hotswap:Hotswap_Choc_V1_1.00u; moved to F.Cu
- moved S11 125.8 mm to (31.5, 96.7), turned to 8 degrees
- moved D11 116.2 mm to (40.4, 95.8), turned to 98 degrees
- moved S12 110.6 mm to (48.4, 84.0), turned to 4 degrees
- moved S13 106.0 mm to (66.6, 75.6)
- moved D12 101.1 mm to (57.4, 83.7), turned to 94 degrees
- moved D13 97.3 mm to (75.5, 76.6), turned to 90 degrees
- moved S6 89.9 mm to (29.1, 79.8), turned to 8 degrees
- moved S7 89.5 mm to (47.3, 67.0), turned to 4 degrees
- moved S14 88.0 mm to (84.6, 81.1)
- moved S1 82.1 mm to (26.8, 63.0)
- moved D7 81.1 mm to (56.2, 67.3), turned to 94 degrees
- moved D6 80.5 mm to (38.1, 79.4), turned to 98 degrees
- moved D14 78.8 mm to (93.5, 82.0), turned to 90 degrees
- moved D1 76.1 mm to (35.8, 62.8), turned to 98 degrees
- moved S15 75.7 mm to (102.6, 83.6)
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Connections:
- net P21 renamed LRow 3
- D1 pad 1: P4 -> LRow 0
- D1 pad 2: pinky_bottom -> Net-(D1-A)
- D10 pad 1: P4 -> LRow 1
- D10 pad 2: index_bottom -> Net-(D10-A)
- D11 pad 1: P3 -> LRow 2
- D11 pad 2: index_home -> Net-(D11-A)
- D12 pad 1: P2 -> LRow 2
- D12 pad 2: index_top -> Net-(D12-A)
- D13 pad 1: P4 -> LRow 2
- D13 pad 2: inner_bottom -> Net-(D13-A)
- D14 pad 1: P3 -> LRow 2
- D14 pad 2: inner_home -> Net-(D14-A)
- D15 pad 1: P2 -> LRow 2
- D15 pad 2: inner_top -> Net-(D15-A)
- D16 pad 2: left_cluster -> Net-(D16-A)
- D17 pad 2: mid_cluster -> Net-(D17-A)
- D18 pad 2: right_cluster -> Net-(D18-A)
- D2 pad 1: P3 -> LRow 0
- D2 pad 2: pinky_home -> Net-(D2-A)
- D3 pad 1: P2 -> LRow 0
- D3 pad 2: pinky_top -> Net-(D3-A)
- D4 pad 1: P4 -> LRow 0
- D4 pad 2: ring_bottom -> Net-(D4-A)
- D5 pad 1: P3 -> LRow 0
- D5 pad 2: ring_home -> Net-(D5-A)
- D6 pad 1: P2 -> LRow 1
- D6 pad 2: ring_top -> Net-(D6-A)
- D7 pad 1: P4 -> LRow 1
- D7 pad 2: middle_bottom -> Net-(D7-A)
- D8 pad 1: P3 -> LRow 1
- D8 pad 2: middle_home -> Net-(D8-A)
- D9 pad 1: P2 -> LRow 1
- D9 pad 2: middle_top -> Net-(D9-A)
- LED1 pad 2: P10 -> unconnected-(LED1-DOUT-Pad2)
- LED1 pad 3: GND -> L_LED_DIN
- LED1 pad 4: LED_1_DOUT -> GND
- LED2 pad 2: LED_1_DOUT -> unconnected-(LED2-DOUT-Pad2)
- LED2 pad 3: GND -> LED1_DIN
- LED2 pad 4: Final -> GND
- S1 pad 1: P5 -> LCol 0
- S1 pad 2: P5 -> Net-(D1-A)
- S10 pad 1: P8 -> LCol 4
- S10 pad 2: P8 -> Net-(D10-A)
- S11 pad 1: P8 -> LCol 0
- S11 pad 2: P8 -> Net-(D11-A)
- S12 pad 1: P8 -> LCol 1
- S12 pad 2: P8 -> Net-(D12-A)
- S13 pad 1: P9 -> LCol 2
- S13 pad 2: P9 -> Net-(D13-A)
- S14 pad 1: P9 -> LCol 3
- S14 pad 2: P9 -> Net-(D14-A)
- S15 pad 1: P9 -> LCol 4
- S15 pad 2: P9 -> Net-(D15-A)
- S16 pad 1: P20 -> LCol 3
- S16 pad 2: P20 -> Net-(D16-A)
- S17 pad 1: P19 -> LCol 4
- S17 pad 2: P19 -> Net-(D17-A)
- S18 pad 1: P18 -> LCol 5
- S18 pad 2: P18 -> Net-(D18-A)
- S2 pad 1: P5 -> LCol 1
- S2 pad 2: P5 -> Net-(D2-A)
- S3 pad 1: P5 -> LCol 2
- S3 pad 2: P5 -> Net-(D3-A)
- S4 pad 1: P6 -> LCol 3
- S4 pad 2: P6 -> Net-(D4-A)
- S5 pad 1: P6 -> LCol 4
- S5 pad 2: P6 -> Net-(D5-A)
- S6 pad 1: P6 -> LCol 0
- S6 pad 2: P6 -> Net-(D6-A)
- S7 pad 1: P7 -> LCol 1
- S7 pad 2: P7 -> Net-(D7-A)
- S8 pad 1: P7 -> LCol 2
- S8 pad 2: P7 -> Net-(D8-A)
- S9 pad 1: P7 -> LCol 3
- S9 pad 2: P7 -> Net-(D9-A)
Routing:
- net LCol 0: track 0.00 -> 186.3 mm
- net Col 0: track 0.00 -> 186.2 mm
- net LCol 1: track 0.00 -> 156.9 mm
- net Col 1: track 0.00 -> 156.4 mm
- net P5: track 150.8 -> 0.00 mm, vias 3 -> 0
- net P6: track 133.6 -> 0.00 mm, vias 3 -> 0
- net Row 2: track 0.00 -> 131.0 mm
- net LCol 3: track 0.00 -> 130.1 mm
- net Col 3: track 0.00 -> 128.2 mm
- net LCol 2: track 0.00 -> 127.9 mm
- net LRow 2: track 0.00 -> 125.7 mm, vias 0 -> 1
- net Col 2: track 0.00 -> 124.3 mm
- net P2: track 123.1 -> 0.00 mm, vias 5 -> 0
- net RST: track 121.0 -> 0.00 mm, vias 3 -> 0
- net Col 4: track 0.00 -> 116.3 mm
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Other:
- board size 131.9 x 104.1 mm -> 251.2 x 101.7 mm
- rule pad_to_mask_clearance: 0.05 -> 0
- board text added: "DRC failed I but I didn't. Yari V1"
- board text added: "Tolerance is a just a suggestion. Yari V1"
- board text removed: "DRC failed but I didn't."
- board text removed: "Tolerance is a suggestion."
- board text removed: "Yari"
- board text removed: "ver 1.0.0"
- board text removed: "{dblquote}Sufficiently advanced bugs are indistinguishable from features.{dblquote}"
